File: ergogen/build/pcbs/scyline_mx.kicad_pcb (KiCad board)
At the start: 2 copper layers, 131.8 x 104.7 mm, 93 parts

Commit message: Build
Parts:
- added J1: qwiik_jst, scybin:qwiik_jst, F.Cu at (218.5, 164.4)
- MCU1: footprint ceoloide:mcu_nice_nano -> scybin:mcu_nice_nano
- moved MCU1 41.9 mm to (214.0, 89.0)
- moved JST1 14.5 mm to (218.5, 149.9), turned to 0 degrees
Connections:
- MCU1 pad 105: P2 -> SDA
- MCU1 pad 106: R0 -> SCL
- MCU1 pad 107: R1 -> R0
- MCU1 pad 108: R2 -> R1
- MCU1 pad 109: R3 -> R2
- MCU1 pad 110: R4 -> R3
- MCU1 pad 111: P8 -> R4
Other:
- outline, holes or cut-outs redrawn

Commit message: Build
Parts:
- added D55: , ceoloide:diode_tht_sod123, F.Cu at (207.3, 155.9)
- added D56: , ceoloide:diode_tht_sod123, F.Cu at (221.8, 136.9)
- added S28: , ceoloide:switch_mx, B.Cu at (214.0, 138.4)
- D28: moved to B.Cu
- moved D28 99.0 mm to (206.2, 136.9)
- moved D52 86.1 mm to (202.8, 79.9), turned to -90 degrees
- moved D44 64.6 mm to (164.8, 72.3)
- moved D48 62.8 mm to (183.8, 77.1)
- moved D32 58.3 mm to (107.8, 91.5)
- moved D40 55.6 mm to (145.8, 77.1)
- moved D36 48.3 mm to (126.8, 89.6)
- moved J1 40.3 mm to (214.0, 124.4)
- moved D54 23.5 mm to (183.8, 155.9)
- moved D53 20.8 mm to (163.0, 156.3), turned to -80 degrees
- moved D29 19.0 mm to (107.8, 148.5)
- moved D30 19.0 mm to (107.8, 129.5)
- moved D31 19.0 mm to (107.8, 110.5)
- moved D33 19.0 mm to (126.8, 146.6)
- moved D34 19.0 mm to (126.8, 127.6)
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Connections:
- D28 pad 2: outer_bottom_B -> macro_bottom_B
- D29 pad 1: R2 -> R3
- D29 pad 2: outer_home_B -> outer_bottom_B
- D30 pad 1: R1 -> R2
- D30 pad 2: outer_upper_B -> outer_home_B
- D31 pad 1: R0 -> R1
- D31 pad 2: outer_top_B -> outer_upper_B
- D32 pad 1: R3 -> R0
- D32 pad 2: pinky_bottom_B -> outer_top_B
- D33 pad 1: R2 -> R3
- D33 pad 2: pinky_home_B -> pinky_bottom_B
- D34 pad 1: R1 -> R2
- D34 pad 2: pinky_upper_B -> pinky_home_B
- D35 pad 1: R0 -> R1
- D35 pad 2: pinky_top_B -> pinky_upper_B
- D36 pad 1: R3 -> R0
- D36 pad 2: ring_bottom_B -> pinky_top_B
- D37 pad 1: R2 -> R3
- D37 pad 2: ring_home_B -> ring_bottom_B
- D38 pad 1: R1 -> R2
- D38 pad 2: ring_upper_B -> ring_home_B
- D39 pad 1: R0 -> R1
- D39 pad 2: ring_top_B -> ring_upper_B
- D40 pad 1: R3 -> R0
- D40 pad 2: middle_bottom_B -> ring_top_B
- D41 pad 1: R2 -> R3
- D41 pad 2: middle_home_B -> middle_bottom_B
- D42 pad 1: R1 -> R2
- D42 pad 2: middle_upper_B -> middle_home_B
- D43 pad 1: R0 -> R1
- D43 pad 2: middle_top_B -> middle_upper_B
- D44 pad 1: R3 -> R0
- D44 pad 2: index_bottom_B -> middle_top_B
- D45 pad 1: R2 -> R3
- D45 pad 2: index_home_B -> index_bottom_B
- D46 pad 1: R1 -> R2
- D46 pad 2: index_upper_B -> index_home_B
- D47 pad 1: R0 -> R1
- D47 pad 2: index_top_B -> index_upper_B
- D48 pad 1: R3 -> R0
- D48 pad 2: inner_bottom_B -> index_top_B
- D49 pad 1: R2 -> R3
- D49 pad 2: inner_home_B -> inner_bottom_B
- D50 pad 1: R1 -> R2
- D50 pad 2: inner_upper_B -> inner_home_B
- D51 pad 1: R0 -> R1
- D51 pad 2: inner_top_B -> inner_upper_B
- D52 pad 1: R4 -> R0
- D52 pad 2: tuck_cluster_B -> inner_top_B
- D53 pad 2: layer_cluster_B -> tuck_cluster_B
- D54 pad 2: space_cluster_B -> layer_cluster_B
- MCU1 pad 121: VCC -> 3V3
Routing:
- net macro_bottom_B: track 0.00 -> 23.1 mm, vias 0 -> 1
- net C5: track 42.3 -> 52.9 mm, vias 4 -> 5
Other:
- board size 131.8 x 104.7 mm -> 133 x 104.7 mm

Commit message: Build
Parts:
- added D57: , ceoloide:diode_tht_sod123, F.Cu at (221.8, 136.9)
- added D58: , ceoloide:diode_tht_sod123, F.Cu at (221.8, 117.9)
- added S29: , ceoloide:switch_mx, B.Cu at (214.0, 119.4)
- D29: moved to B.Cu
- moved D29 102.9 mm to (206.2, 117.9)
- moved D53 86.1 mm to (202.8, 79.9), turned to -90 degrees
- moved D45 64.6 mm to (164.8, 72.3)
- moved D49 62.8 mm to (183.8, 77.1)
- moved D33 58.3 mm to (107.8, 91.5)
- moved D41 55.6 mm to (145.8, 77.1)
- moved D37 48.3 mm to (126.8, 89.6)
- moved D56 23.9 mm to (207.3, 155.9)
- moved D55 23.5 mm to (183.8, 155.9)
- moved D54 20.8 mm to (163.0, 156.3), turned to -80 degrees
- moved D30 19.0 mm to (107.8, 148.5)
- moved D31 19.0 mm to (107.8, 129.5)
- moved D32 19.0 mm to (107.8, 110.5)
- moved D34 19.0 mm to (126.8, 146.6)
- moved D35 19.0 mm to (126.8, 127.6)
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Connections:
- D29 pad 1: R3 -> R2
- D29 pad 2: outer_bottom_B -> macro_home_B
- D30 pad 1: R2 -> R3
- D30 pad 2: outer_home_B -> outer_bottom_B
- D31 pad 1: R1 -> R2
- D31 pad 2: outer_upper_B -> outer_home_B
- D32 pad 1: R0 -> R1
- D32 pad 2: outer_top_B -> outer_upper_B
- D33 pad 1: R3 -> R0
- D33 pad 2: pinky_bottom_B -> outer_top_B
- D34 pad 1: R2 -> R3
- D34 pad 2: pinky_home_B -> pinky_bottom_B
- D35 pad 1: R1 -> R2
- D35 pad 2: pinky_upper_B -> pinky_home_B
- D36 pad 1: R0 -> R1
- D36 pad 2: pinky_top_B -> pinky_upper_B
- D37 pad 1: R3 -> R0
- D37 pad 2: ring_bottom_B -> pinky_top_B
- D38 pad 1: R2 -> R3
- D38 pad 2: ring_home_B -> ring_bottom_B
- D39 pad 1: R1 -> R2
- D39 pad 2: ring_upper_B -> ring_home_B
- D40 pad 1: R0 -> R1
- D40 pad 2: ring_top_B -> ring_upper_B
- D41 pad 1: R3 -> R0
- D41 pad 2: middle_bottom_B -> ring_top_B
- D42 pad 1: R2 -> R3
- D42 pad 2: middle_home_B -> middle_bottom_B
- D43 pad 1: R1 -> R2
- D43 pad 2: middle_upper_B -> middle_home_B
- D44 pad 1: R0 -> R1
- D44 pad 2: middle_top_B -> middle_upper_B
- D45 pad 1: R3 -> R0
- D45 pad 2: index_bottom_B -> middle_top_B
- D46 pad 1: R2 -> R3
- D46 pad 2: index_home_B -> index_bottom_B
- D47 pad 1: R1 -> R2
- D47 pad 2: index_upper_B -> index_home_B
- D48 pad 1: R0 -> R1
- D48 pad 2: index_top_B -> index_upper_B
- D49 pad 1: R3 -> R0
- D49 pad 2: inner_bottom_B -> index_top_B
- D50 pad 1: R2 -> R3
- D50 pad 2: inner_home_B -> inner_bottom_B
- D51 pad 1: R1 -> R2
- D51 pad 2: inner_upper_B -> inner_home_B
- D52 pad 1: R0 -> R1
- D52 pad 2: inner_top_B -> inner_upper_B
- D53 pad 1: R4 -> R0
- D53 pad 2: tuck_cluster_B -> inner_top_B
- D54 pad 2: layer_cluster_B -> tuck_cluster_B
- D55 pad 2: space_cluster_B -> layer_cluster_B
- D56 pad 1: R3 -> R4
- D56 pad 2: macro_bottom_B -> space_cluster_B
- MCU1 pad 114: P16 -> C6
- S28 pad 1: C5 -> C6
Routing:
- net macro_home_B: track 0.00 -> 23.1 mm, vias 0 -> 1
- net C6: track 0.00 -> 21.2 mm, vias 0 -> 2
- net C5: track 52.9 -> 42.3 mm, vias 5 -> 4

Commit message: Build
Parts:
- turned J1 to 0 degrees
Changed lines of the file:
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@@
   (title_block
     (title "scyline_mx")
-    (date "2025-12-20")
+    (date "2025-12-24")
     (rev "1")
     (company "Scybin")
@@
     (footprint "scybin:qwiik_jst"
       (layer "F.Cu")
-      (at 214 112.41 180)
+      (at 214 112.41 0)
       (descr "JST SH series connector, SM04B-SRSS-TB (http://www.jst-mfg.com/product/pdf/eng/eSH.pdf)")
       (tags "connector JST SH horizontal")
       (property "Reference" "J1"
-        (at 0 -3.98 180)
+        (at 0 -3.98 0)
         (layer "F.SilkS")
         hide
@@
       )
       (property "Value" "qwiik_jst"
-        (at 0 3.98 180)
+        (at 0 3.98 0)
         (layer "F.Fab")
         (effects
@@
       )
       (fp_text user "J1"
-        (at 0 0 180)
+        (at 0 0 0)
         (layer "F.Fab")
         (effects
@@
       )
       (pad "1" smd roundrect
-        (at -1.5 -2 180)
+        (at -1.5 -2 0)
         (size 0.6 1.55)
         (layers "F.Cu" "F.Mask" "F.Paste")
@@
       )
       (pad "2" smd roundrect
-        (at -0.5 -2 180)
+        (at -0.5 -2 0)
         (size 0.6 1.55)
         (layers "F.Cu" "F.Mask" "F.Paste")
@@
       )
       (pad "3" smd roundrect
-        (at 0.5 -2 180)
+        (at 0.5 -2 0)
         (size 0.6 1.55)
         (layers "F.Cu" "F.Mask" "F.Paste")
@@
       )
       (pad "4" smd roundrect
-        (at 1.5 -2 180)
+        (at 1.5 -2 0)
         (size 0.6 1.55)
         (layers "F.Cu" "F.Mask" "F.Paste")
@@
       )
       (pad "MP" smd roundrect
-        (at -2.8 1.875 180)
+        (at -2.8 1.875 0)
         (size 1.2 1.8)
         (layers "F.Cu" "F.Mask" "F.Paste")
@@
       )
       (pad "MP" smd roundrect
-        (at 2.8 1.875 180)
+        (at 2.8 1.875 0)
         (size 1.2 1.8)
         (layers "F.Cu" "F.Mask" "F.Paste")
@@
       )
       (pad "1" smd roundrect
-        (at -1.5 -2 180)
+        (at -1.5 -2 0)
         (size 0.6 1.55)
         (layers "B.Cu" "B.Mask" "B.Paste")
@@
       )
       (pad "2" smd roundrect
-        (at -0.5 -2 180)
+        (at -0.5 -2 0)
         (size 0.6 1.55)
         (layers "B.Cu" "B.Mask" "B.Paste")
@@
       )
       (pad "3" smd roundrect
-        (at 0.5 -2 180)
+        (at 0.5 -2 0)
         (size 0.6 1.55)
         (layers "B.Cu" "B.Mask" "B.Paste")
@@
       )
       (pad "4" smd roundrect
-        (at 1.5 -2 180)
+        (at 1.5 -2 0)
         (size 0.6 1.55)
         (layers "B.Cu" "B.Mask" "B.Paste")
@@
       )
       (pad "MP" smd roundrect
-        (at -2.8 1.875 180)
+        (at -2.8 1.875 0)
         (size 1.2 1.8)
         (layers "B.Cu" "B.Mask" "B.Paste")
@@
       )
       (pad "MP" smd roundrect
-        (at 2.8 1.875 180)
+        (at 2.8 1.875 0)
         (size 1.2 1.8)
         (layers "B.Cu" "B.Mask" "B.Paste")

Commit message: Build
Parts:
- added MH8: , ceoloide:mounting_hole_npth, F.Cu at (204.5, 128.9)
- added MH9: , ceoloide:mounting_hole_npth, F.Cu at (204.5, 147.4)
Connections:
- MCU1 pad 107: R0 -> P4
- MCU1 pad 108: R1 -> R0
- MCU1 pad 109: R2 -> R1
- MCU1 pad 110: R3 -> R2
- MCU1 pad 111: R4 -> R3
- MCU1 pad 112: P9 -> R4
Other:
- outline, holes or cut-outs redrawn

Commit message: Build
Parts:
- J1: footprint scybin:qwiik_jst -> scyline:qwiik_jst
- JST1: footprint ceoloide:battery_connector_jst_ph_2 -> scyline:battery_connector_jst_ph_2
- LOGO1: footprint ceoloide:utility_ergogen_logo -> scyline:utility_ergogen_logo
- MCU1: footprint scybin:mcu_nice_nano -> scyline:mcu_nice_nano_4mm
- PWR1: footprint ceoloide:power_switch_smd_side -> scyline:power_switch_smd_side
- RST1: footprint ceoloide:reset_switch_smd_side -> scyline:reset_switch_smd_side
- S1, S10, S11, S12, S13, S14, S15, S16, S17, S18, S19, S2, S20, S21, S22, S23, S24, S25, S26, S27, S28, S3, S4, S5, S6, S7, S8, S9: footprint ceoloide:switch_mx -> scyline:scybin_switch_mx
Connections:
- PWR1 pad 3: BAT_P -> (no net)
Routing:
- net (no net): track 333.1 -> 0.00 mm
- net C2: track 52.9 -> 111.8 mm
- net C3: track 52.9 -> 111.8 mm
- net C4: track 52.9 -> 111.8 mm
- net C5: track 42.3 -> 91.4 mm
- net C1: track 42.3 -> 91.4 mm
- net C0: track 42.3 -> 91.4 mm
- net C6: track 21.2 -> 50.5 mm
- net GND: track 0.00 -> 28.9 mm
- net tuck_cluster_B: track 23.1 -> 13.2 mm
- net space_cluster_B: track 23.1 -> 13.2 mm
- net macro_bottom_B: track 23.1 -> 13.2 mm
- net layer_cluster_B: track 23.1 -> 13.2 mm
- net inner_bottom_B: track 23.1 -> 13.2 mm
- net pinky_home_B: track 23.1 -> 13.2 mm
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
Commit message: Build
Parts:
- J1: footprint scyline:qwiik_jst -> scybin:qwiik_jst
- JST1: footprint scyline:battery_connector_jst_ph_2 -> ceoloide:battery_connector_jst_ph_2
- LOGO1: footprint scyline:utility_ergogen_logo -> ceoloide:utility_ergogen_logo
- MCU1: footprint scyline:mcu_nice_nano_4mm -> scybin:mcu_nice_nano
- PWR1: footprint scyline:power_switch_smd_side -> ceoloide:power_switch_smd_side
- RST1: footprint scyline:reset_switch_smd_side -> ceoloide:reset_switch_smd_side
- S1, S10, S11, S12, S13, S14, S15, S16, S17, S18, S19, S2, S20, S21, S22, S23, S24, S25, S26, S27, S28, S3, S4, S5, S6, S7, S8, S9: footprint scyline:scybin_switch_mx -> ceoloide:switch_mx
Connections:
- PWR1 pad 3: (no net) -> BAT_P
Routing:
- net (no net): track 0.00 -> 333.1 mm
- net C2: track 111.8 -> 52.9 mm
- net C3: track 111.8 -> 52.9 mm
- net C4: track 111.8 -> 52.9 mm
- net C5: track 91.4 -> 42.3 mm
- net C1: track 91.4 -> 42.3 mm
- net C0: track 91.4 -> 42.3 mm
- net C6: track 50.5 -> 21.2 mm
- net GND: track 28.9 -> 0.00 mm
- net tuck_cluster_B: track 13.2 -> 23.1 mm
- net space_cluster_B: track 13.2 -> 23.1 mm
- net macro_bottom_B: track 13.2 -> 23.1 mm
- net layer_cluster_B: track 13.2 -> 23.1 mm
- net inner_bottom_B: track 13.2 -> 23.1 mm
- net pinky_home_B: track 13.2 -> 23.1 mm
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Other:
- outline, holes or cut-outs redrawn

Commit message: Build
Parts:
- moved J1 3.30 mm to (214.0, 109.1)
Changed lines of the file:
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@@
     (footprint "scybin:qwiik_jst"
       (layer "F.Cu")
-      (at 214 112.41 0)
+      (at 214 109.11 0)
       (descr "JST SH series connector, SM04B-SRSS-TB (http://www.jst-mfg.com/product/pdf/eng/eSH.pdf)")
       (tags "connector JST SH horizontal")
