File: ergogen/build/pcbs/scyline_mx.kicad_pcb (KiCad board)
At the start: 2 copper layers, 133 x 104.7 mm, 102 parts, among them J1 qwiik_jst

Commit message: Build
Parts:
- moved D49 106.1 mm to (100.0, 142.0), turned to 180 degrees
- moved D7 104.6 mm to (214.0, 127.9), turned to 180 degrees
- moved D20 94.1 mm to (100.0, 142.0), turned to 180 degrees
- moved D6 91.9 mm to (195.0, 89.9), turned to 180 degrees
- moved D36 89.3 mm to (214.0, 127.9), turned to 180 degrees
- moved D5 88.0 mm to (176.0, 87.1), turned to 180 degrees
- moved D50 83.9 mm to (119.0, 140.1), turned to 180 degrees
- moved D35 77.9 mm to (195.0, 89.9), turned to 180 degrees
- moved D34 77.2 mm to (176.0, 87.1), turned to 180 degrees
- moved D43 71.1 mm to (100.0, 139.5), turned to 180 degrees
- moved D21 68.2 mm to (119.0, 140.1), turned to 180 degrees
- moved D51 65.6 mm to (138.0, 127.6), turned to 180 degrees
- moved D4 65.5 mm to (157.0, 82.3), turned to 180 degrees
- moved D44 65.2 mm to (119.0, 137.6), turned to 180 degrees
- moved D45 59.2 mm to (138.0, 125.1), turned to 180 degrees
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Connections:
- D1 pad 1: R3 -> R0
- D1 pad 2: outer_bottom_B -> outer_top_B
- D10 pad 1: R2 -> R1
- D10 pad 2: ring_home_B -> ring_upper_B
- D11 pad 2: ring_upper_B -> middle_upper_B
- D12 pad 1: R0 -> R1
- D12 pad 2: ring_top_B -> index_upper_B
- D13 pad 1: R3 -> R1
- D13 pad 2: middle_bottom_B -> inner_upper_B
- D14 pad 2: middle_home_B -> outer_home_B
- D15 pad 1: R1 -> R2
- D15 pad 2: middle_upper_B -> pinky_home_B
- D16 pad 1: R0 -> R2
- D16 pad 2: middle_top_B -> ring_home_B
- D17 pad 1: R3 -> R2
- D17 pad 2: index_bottom_B -> middle_home_B
- D19 pad 1: R1 -> R2
- D19 pad 2: index_upper_B -> inner_home_B
- D2 pad 1: R2 -> R0
- D2 pad 2: outer_home_B -> pinky_top_B
- D20 pad 1: R0 -> R3
- D20 pad 2: index_top_B -> outer_bottom_B
- D21 pad 2: inner_bottom_B -> pinky_bottom_B
- D22 pad 1: R2 -> R3
- D22 pad 2: inner_home_B -> ring_bottom_B
- D23 pad 1: R1 -> R3
- D23 pad 2: inner_upper_B -> middle_bottom_B
- D24 pad 1: R0 -> R3
- D24 pad 2: inner_top_B -> index_bottom_B
- D25 pad 1: R4 -> R3
- D25 pad 2: tuck_cluster_B -> inner_bottom_B
- D26 pad 1: R4 -> R3
- D26 pad 2: layer_cluster_B -> macro_bottom_B
- D27 pad 2: space_cluster_B -> tuck_cluster_B
- D28 pad 1: R3 -> R4
- D28 pad 2: macro_bottom_B -> layer_cluster_B
- D29 pad 1: R2 -> R4
- D29 pad 2: macro_home_B -> space_cluster_B
- D3 pad 1: R1 -> R0
- D3 pad 2: outer_upper_B -> ring_top_B
- D30 pad 1: R3 -> R0
- D30 pad 2: outer_bottom_B -> outer_top_B
- D31 pad 1: R2 -> R0
- D31 pad 2: outer_home_B -> pinky_top_B
- D32 pad 1: R1 -> R0
- D32 pad 2: outer_upper_B -> ring_top_B
- D33 pad 2: outer_top_B -> middle_top_B
- D34 pad 1: R3 -> R0
- D34 pad 2: pinky_bottom_B -> index_top_B
- D35 pad 1: R2 -> R0
- D35 pad 2: pinky_home_B -> inner_top_B
- D36 pad 1: R1 -> R2
- D36 pad 2: pinky_upper_B -> macro_home_B
- D37 pad 1: R0 -> R1
- D37 pad 2: pinky_top_B -> outer_upper_B
- D38 pad 1: R3 -> R1
- D38 pad 2: ring_bottom_B -> pinky_upper_B
- D39 pad 1: R2 -> R1
- D39 pad 2: ring_home_B -> ring_upper_B
- D4 pad 2: outer_top_B -> middle_top_B
- D40 pad 2: ring_upper_B -> middle_upper_B
- D41 pad 1: R0 -> R1
- D41 pad 2: ring_top_B -> index_upper_B
- D42 pad 1: R3 -> R1
- D42 pad 2: middle_bottom_B -> inner_upper_B
- D43 pad 2: middle_home_B -> outer_home_B
- D44 pad 1: R1 -> R2
- D44 pad 2: middle_upper_B -> pinky_home_B
- D45 pad 1: R0 -> R2
- D45 pad 2: middle_top_B -> ring_home_B
- D46 pad 1: R3 -> R2
- D46 pad 2: index_bottom_B -> middle_home_B
- D48 pad 1: R1 -> R2
- D48 pad 2: index_upper_B -> inner_home_B
- D49 pad 1: R0 -> R3
- D49 pad 2: index_top_B -> outer_bottom_B
- D5 pad 1: R3 -> R0
- D5 pad 2: pinky_bottom_B -> index_top_B
- D50 pad 2: inner_bottom_B -> pinky_bottom_B
- D51 pad 1: R2 -> R3
- D51 pad 2: inner_home_B -> ring_bottom_B
- D52 pad 1: R1 -> R3
- D52 pad 2: inner_upper_B -> middle_bottom_B
- D53 pad 1: R0 -> R3
- D53 pad 2: inner_top_B -> index_bottom_B
- D54 pad 1: R4 -> R3
- D54 pad 2: tuck_cluster_B -> inner_bottom_B
- D55 pad 1: R4 -> R3
- D55 pad 2: layer_cluster_B -> macro_bottom_B
- D56 pad 2: space_cluster_B -> tuck_cluster_B
- D57 pad 1: R3 -> R4
- D57 pad 2: macro_bottom_B -> layer_cluster_B
- D58 pad 1: R2 -> R4
- D58 pad 2: macro_home_B -> space_cluster_B
- D6 pad 1: R2 -> R0
- D6 pad 2: pinky_home_B -> inner_top_B
- D7 pad 1: R1 -> R2
- D7 pad 2: pinky_upper_B -> macro_home_B
- D8 pad 1: R0 -> R1
- D8 pad 2: pinky_top_B -> outer_upper_B
- D9 pad 1: R3 -> R1
- D9 pad 2: ring_bottom_B -> pinky_upper_B

Commit message: Build
Parts:
- moved D49 106.1 mm to (183.8, 77.1), turned to -90 degrees
- moved D7 104.6 mm to (111.2, 108.6), turned to -90 degrees
- moved D20 94.1 mm to (168.2, 77.1), turned to -90 degrees
- moved D6 91.9 mm to (111.2, 127.6), turned to -90 degrees
- moved D36 89.3 mm to (126.8, 108.6), turned to -90 degrees
- moved D5 88.0 mm to (111.2, 146.6), turned to -90 degrees
- moved D50 83.9 mm to (202.8, 136.9), turned to -90 degrees
- moved D35 77.9 mm to (126.8, 127.6), turned to -90 degrees
- moved D34 77.2 mm to (126.8, 146.6), turned to -90 degrees
- moved D43 71.1 mm to (164.8, 110.3), turned to -90 degrees
- moved D21 68.2 mm to (187.2, 136.9), turned to -90 degrees
- moved D51 65.6 mm to (202.8, 117.9), turned to -90 degrees
- moved D4 65.5 mm to (92.2, 91.5), turned to -90 degrees
- moved D44 65.2 mm to (164.8, 91.3), turned to -90 degrees
- moved D45 59.2 mm to (164.8, 72.3), turned to -90 degrees
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Connections:
- D1 pad 1: R0 -> R3
- D1 pad 2: outer_top_B -> outer_bottom_B
- D10 pad 1: R1 -> R2
- D10 pad 2: ring_upper_B -> ring_home_B
- D11 pad 2: middle_upper_B -> ring_upper_B
- D12 pad 1: R1 -> R0
- D12 pad 2: index_upper_B -> ring_top_B
- D13 pad 1: R1 -> R3
- D13 pad 2: inner_upper_B -> middle_bottom_B
- D14 pad 2: outer_home_B -> middle_home_B
- D15 pad 1: R2 -> R1
- D15 pad 2: pinky_home_B -> middle_upper_B
- D16 pad 1: R2 -> R0
- D16 pad 2: ring_home_B -> middle_top_B
- D17 pad 1: R2 -> R3
- D17 pad 2: middle_home_B -> index_bottom_B
- D19 pad 1: R2 -> R1
- D19 pad 2: inner_home_B -> index_upper_B
- D2 pad 1: R0 -> R2
- D2 pad 2: pinky_top_B -> outer_home_B
- D20 pad 1: R3 -> R0
- D20 pad 2: outer_bottom_B -> index_top_B
- D21 pad 2: pinky_bottom_B -> inner_bottom_B
- D22 pad 1: R3 -> R2
- D22 pad 2: ring_bottom_B -> inner_home_B
- D23 pad 1: R3 -> R1
- D23 pad 2: middle_bottom_B -> inner_upper_B
- D24 pad 1: R3 -> R0
- D24 pad 2: index_bottom_B -> inner_top_B
- D25 pad 1: R3 -> R4
- D25 pad 2: inner_bottom_B -> tuck_cluster_B
- D26 pad 1: R3 -> R4
- D26 pad 2: macro_bottom_B -> layer_cluster_B
- D27 pad 2: tuck_cluster_B -> space_cluster_B
- D28 pad 1: R4 -> R3
- D28 pad 2: layer_cluster_B -> macro_bottom_B
- D29 pad 1: R4 -> R2
- D29 pad 2: space_cluster_B -> macro_home_B
- D3 pad 1: R0 -> R1
- D3 pad 2: ring_top_B -> outer_upper_B
- D30 pad 1: R0 -> R3
- D30 pad 2: outer_top_B -> outer_bottom_B
- D31 pad 1: R0 -> R2
- D31 pad 2: pinky_top_B -> outer_home_B
- D32 pad 1: R0 -> R1
- D32 pad 2: ring_top_B -> outer_upper_B
- D33 pad 2: middle_top_B -> outer_top_B
- D34 pad 1: R0 -> R3
- D34 pad 2: index_top_B -> pinky_bottom_B
- D35 pad 1: R0 -> R2
- D35 pad 2: inner_top_B -> pinky_home_B
- D36 pad 1: R2 -> R1
- D36 pad 2: macro_home_B -> pinky_upper_B
- D37 pad 1: R1 -> R0
- D37 pad 2: outer_upper_B -> pinky_top_B
- D38 pad 1: R1 -> R3
- D38 pad 2: pinky_upper_B -> ring_bottom_B
- D39 pad 1: R1 -> R2
- D39 pad 2: ring_upper_B -> ring_home_B
- D4 pad 2: middle_top_B -> outer_top_B
- D40 pad 2: middle_upper_B -> ring_upper_B
- D41 pad 1: R1 -> R0
- D41 pad 2: index_upper_B -> ring_top_B
- D42 pad 1: R1 -> R3
- D42 pad 2: inner_upper_B -> middle_bottom_B
- D43 pad 2: outer_home_B -> middle_home_B
- D44 pad 1: R2 -> R1
- D44 pad 2: pinky_home_B -> middle_upper_B
- D45 pad 1: R2 -> R0
- D45 pad 2: ring_home_B -> middle_top_B
- D46 pad 1: R2 -> R3
- D46 pad 2: middle_home_B -> index_bottom_B
- D48 pad 1: R2 -> R1
- D48 pad 2: inner_home_B -> index_upper_B
- D49 pad 1: R3 -> R0
- D49 pad 2: outer_bottom_B -> index_top_B
- D5 pad 1: R0 -> R3
- D5 pad 2: index_top_B -> pinky_bottom_B
- D50 pad 2: pinky_bottom_B -> inner_bottom_B
- D51 pad 1: R3 -> R2
- D51 pad 2: ring_bottom_B -> inner_home_B
- D52 pad 1: R3 -> R1
- D52 pad 2: middle_bottom_B -> inner_upper_B
- D53 pad 1: R3 -> R0
- D53 pad 2: index_bottom_B -> inner_top_B
- D54 pad 1: R3 -> R4
- D54 pad 2: inner_bottom_B -> tuck_cluster_B
- D55 pad 1: R3 -> R4
- D55 pad 2: macro_bottom_B -> layer_cluster_B
- D56 pad 2: tuck_cluster_B -> space_cluster_B
- D57 pad 1: R4 -> R3
- D57 pad 2: layer_cluster_B -> macro_bottom_B
- D58 pad 1: R4 -> R2
- D58 pad 2: space_cluster_B -> macro_home_B
- D6 pad 1: R0 -> R2
- D6 pad 2: inner_top_B -> pinky_home_B
- D7 pad 1: R2 -> R1
- D7 pad 2: macro_home_B -> pinky_upper_B
- D8 pad 1: R1 -> R0
- D8 pad 2: outer_upper_B -> pinky_top_B
- D9 pad 1: R1 -> R3
- D9 pad 2: pinky_upper_B -> ring_bottom_B
Other:
- board size 133 x 104.7 mm -> 134 x 106.7 mm

Commit message: Build
Connections:
- net 3V3 renamed V+
Changed lines of the file:
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@@
 (net 45 "RAW")
 (net 46 "RST")
-(net 47 "3V3")
+(net 47 "V+")
 (net 48 "P10")
 (net 49 "P1")
@@
     (pad "21" thru_hole circle (at -7.62 -5.079999999999999 0) (size 1.7 1.7) (drill 0.85) (layers "*.Cu" "*.Mask") (net 63 "MCU1_21"))
     (pad "4" thru_hole circle (at 7.62 -5.079999999999999 0) (size 1.7 1.7) (drill 0.85) (layers "*.Cu" "*.Mask") (net 64 "MCU1_4"))
-    (pad "121" thru_hole circle (at -3.4 -5.079999999999999 0) (size 0.8 0.8) (drill 0.4) (layers "*.Cu" "*.Mask") (net 47 "3V3"))
+    (pad "121" thru_hole circle (at -3.4 -5.079999999999999 0) (size 0.8 0.8) (drill 0.4) (layers "*.Cu" "*.Mask") (net 47 "V+"))
     (pad "104" thru_hole circle (at 3.4 -5.079999999999999 0) (size 0.8 0.8) (drill 0.4) (layers "*.Cu" "*.Mask") (net 3 "GND"))
     (pad "21" smd rect (at -5.48 -5.079999999999999 0) (size 0.6 1.2) (layers "F.Cu" "F.Paste" "F.Mask") (net 63 "MCU1_21"))
-    (pad "121" smd rect (at -4.58 -5.079999999999999 0) (size 0.6 1.2) (layers "F.Cu" "F.Paste" "F.Mask") (net 47 "3V3"))
+    (pad "121" smd rect (at -4.58 -5.079999999999999 0) (size 0.6 1.2) (layers "F.Cu" "F.Paste" "F.Mask") (net 47 "V+"))
     (pad "104" smd rect (at 4.58 -5.079999999999999 0) (size 0.6 1.2) (layers "F.Cu" "F.Paste" "F.Mask") (net 3 "GND"))
     (pad "4" smd rect (at 5.48 -5.079999999999999 0) (size 0.6 1.2) (layers "F.Cu" "F.Paste" "F.Mask") (net 64 "MCU1_4"))
     (pad "21" smd rect (at -5.48 -5.079999999999999 0) (size 0.6 1.2) (layers "B.Cu" "B.Paste" "B.Mask") (net 63 "MCU1_21"))
     (pad "104" smd rect (at -4.58 -5.079999999999999 0) (size 0.6 1.2) (layers "B.Cu" "B.Paste" "B.Mask") (net 3 "GND"))
-    (pad "121" smd rect (at 4.58 -5.079999999999999 0) (size 0.6 1.2) (layers "B.Cu" "B.Paste" "B.Mask") (net 47 "3V3"))
+    (pad "121" smd rect (at 4.58 -5.079999999999999 0) (size 0.6 1.2) (layers "B.Cu" "B.Paste" "B.Mask") (net 47 "V+"))
     (pad "4" smd rect (at 5.48 -5.079999999999999 0) (size 0.6 1.2) (layers "B.Cu" "B.Paste" "B.Mask") (net 64 "MCU1_4"))
-    (fp_text user "3V3" (at -1.45 -5.079999999999999 0) (layer "F.SilkS")
+    (fp_text user "V+" (at -2.04 -5.079999999999999 0) (layer "F.SilkS")
       (effects (font (size 1 1) (thickness 0.15)))
     )
@@
       (effects (font (size 1 1) (thickness 0.15)) (justify mirror))
     )
-    (fp_text user "3V3" (at 1.45 -5.079999999999999 0) (layer "B.SilkS")
+    (fp_text user "V+" (at 2.04 -5.079999999999999 0) (layer "B.SilkS")
       (effects (font (size 1 1) (thickness 0.15)) (justify mirror))
     )
-    (fp_text user "3V3" (at -3.262 -5.88 0) (layer "F.Fab")
+    (fp_text user "V+" (at -3.262 -5.88 0) (layer "F.Fab")
       (effects (font (size 0.5 0.5) (thickness 0.08)))
     )
@@
       (effects (font (size 0.5 0.5) (thickness 0.08)))
     )
-    (fp_text user "3V3" (at -3.262 -5.88 180) (layer "B.Fab")
+    (fp_text user "V+" (at -3.262 -5.88 180) (layer "B.Fab")
       (effects (font (size 0.5 0.5) (thickness 0.08)) (justify mirror))
     )
@@
         (layers "F.Cu" "F.Mask" "F.Paste")
         (roundrect_rratio 0.25)
-        (net 47 "3V3")
+        (net 47 "V+")
       )
       (pad "3" smd roundrect
@@
         (layers "B.Cu" "B.Mask" "B.Paste")
         (roundrect_rratio 0.25)
-        (net 47 "3V3")
+        (net 47 "V+")
       )
       (pad "3" smd roundrect

Commit message: Build
Parts:
- moved PWR1 0.20 mm to (142.0, 164.3)
