File: ergogen/build/pcbs/_autosave-scyline_mx.kicad_pcb (KiCad board)
At the start: 2 copper layers, 133 x 104.7 mm, 102 parts, among them J1 qwiik_jst

Commit message: Build
Parts:
- S1, S10, S11, S12, S13, S14, S15, S16, S17, S18, S19, S2, S20, S21, S22, S23, S24, S25, S26, S27, S28, S3, S4, S5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: footprint scyline:scybin_switch_mx -> ceoloide:switch_mx
