File: ergogen/build/pcbs/_autosave-scyline_mx.kicad_pcb (KiCad board)
At the start: 2 copper layers, 134 x 106.7 mm, 102 parts, among them J1 qwiik_jst

Commit message: Build
Parts:
- D1, D10, D11, D12, D13, D14, D15, D16, D17, D18, D19, D2, D20, D21, D22, D23, D24, D25, D26, D27, D28, D29, D3, D30, D31, D32, D33, D34, D35, D36, D37, D38, D39, D4, D40, D41, D42, D43, D44, D45, D46, D47, D48, D49, D5, D50, D51, D52, D53, D54, D55, D56, D57, D58, D6, D7, D8, D9: footprint scyline:diode_tht_sod123 -> ceoloide:diode_tht_sod123
- JST1: footprint scyline:battery_connector_jst_ph_2 -> ceoloide:battery_connector_jst_ph_2
- PWR1: footprint scyline:power_switch_smd_side -> ceoloide:power_switch_smd_side
- RST1: footprint scyline:reset_switch_smd_side -> ceoloide:reset_switch_smd_side
- S1, S10, S11, S12, S13, S14, S15, S16, S17, S18, S19, S2, S20, S21, S22, S23, S24, S25, S26, S27, S28, S3, S4, S5, S6, S7, S8, S9: footprint scyline:scybin_switch_mx -> ceoloide:switch_mx
- moved PWR1 0.20 mm to (142.0, 164.3)
Connections:
- net 3V3 renamed V+
- PWR1 pad 3: (no net) -> BAT_P
