File: ergogen/build/pcbs/chitin.kicad_pcb (KiCad board)
At the start: 2 copper layers, 134 x 106.7 mm, 102 parts, among them J1 qwiik_jst

Commit message: Build
Parts:
- added MH10: , ceoloide:mounting_hole_npth, F.Cu at (138.0, 116.6)
- added MH11: , ceoloide:mounting_hole_npth, F.Cu at (138.0, 97.6)
- added MH12: , ceoloide:mounting_hole_npth, F.Cu at (138.0, 78.6)
- added MH13: , ceoloide:mounting_hole_npth, F.Cu at (157.0, 130.8)
- added MH14: , ceoloide:mounting_hole_npth, F.Cu at (157.0, 111.8)
- added MH15: , ceoloide:mounting_hole_npth, F.Cu at (157.0, 92.8)
- added MH16: , ceoloide:mounting_hole_npth, F.Cu at (157.0, 73.8)
- added MH17: , ceoloide:mounting_hole_npth, F.Cu at (176.0, 135.6)
- added MH18: , ceoloide:mounting_hole_npth, F.Cu at (176.0, 116.6)
- added MH19: , ceoloide:mounting_hole_npth, F.Cu at (176.0, 97.6)
- added MH20: , ceoloide:mounting_hole_npth, F.Cu at (176.0, 78.6)
- added MH21: , ceoloide:mounting_hole_npth, F.Cu at (195.0, 138.4)
- added MH22: , ceoloide:mounting_hole_npth, F.Cu at (195.0, 119.4)
- added MH23: , ceoloide:mounting_hole_npth, F.Cu at (195.0, 100.4)
- added MH24: , ceoloide:mounting_hole_npth, F.Cu at (195.0, 81.4)
- added MH25: , ceoloide:mounting_hole_npth, F.Cu at (155.6, 159.1)
- added MH26: , ceoloide:mounting_hole_npth, F.Cu at (176.0, 157.4)
- added MH27: , ceoloide:mounting_hole_npth, F.Cu at (199.5, 157.4)
- added MH28: , ceoloide:mounting_hole_npth, F.Cu at (214.0, 138.4)
- added MH29: , ceoloide:mounting_hole_npth, F.Cu at (214.0, 119.4)
- moved MH8 93.5 mm to (119.0, 91.1)
- moved MH5 88.6 mm to (119.0, 148.1)
- moved MH4 76.6 mm to (100.0, 93.0)
- moved MH6 69.6 mm to (119.0, 129.1)
- moved MH7 68.7 mm to (119.0, 110.1)
- moved MH9 67.5 mm to (138.0, 135.6)
- moved MH1 49.4 mm to (100.0, 150.0)
- moved MH3 29.1 mm to (100.0, 112.0)
- moved MH2 14.1 mm to (100.0, 131.0)

Commit message: Build
Parts:
- LOGO1: footprint logo_dual -> logo_dual_chitin
Changed lines of the file:
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@@
       )
     )
-(footprint "logo_dual"
+(footprint "logo_dual_chitin"
 	(layer "F.Cu")
 	(at 147 115.85 0)
@@
 	)
 	(attr board_only exclude_from_pos_files exclude_from_bom)
+	(fp_text user "chitin"
+		(at 55 34 0)
+		(layer "F.SilkS")
+		(effects
+			(font
+				(size 2 2)
+				(thickness 0.25)
+			)
+		)
+	)
+	(fp_text user "chitin"
+		(at 55 34 0)
+		(layer "B.SilkS")
+		(effects
+			(font
+				(size 2 2)
+				(thickness 0.25)
+			)
+			(justify mirror)
+		)
+	)
 	(fp_poly
 			(pts
@@
 			(layer "B.SilkS")
 		)
+	(embedded_fonts no)
 )
   (footprint "ceoloide:mounting_hole_npth"

Commit message: Build
Parts:
- removed MH10, MH11, MH12, MH13, MH14, MH15, MH16, MH17, MH18, MH19, MH20, MH21, MH22, MH23, MH24, MH25, MH26, MH27, MH28, MH29: , ceoloide:mounting_hole_npth
- moved MH8 93.5 mm to (204.5, 128.9)
- moved MH5 88.6 mm to (185.5, 89.5)
- moved MH4 76.6 mm to (156.3, 145.0)
- moved MH6 69.6 mm to (185.5, 108.5)
- moved MH7 68.7 mm to (185.5, 127.5)
- moved MH9 67.5 mm to (204.5, 147.4)
- moved MH1 49.4 mm to (109.5, 101.5)
- moved MH3 29.1 mm to (109.5, 139.6)
- moved MH2 14.1 mm to (109.5, 120.5)
