File: kicad/chitin.kicad_pcb (KiCad board)
At the start: 2 copper layers, 134 x 106.7 mm, 102 parts, among them J1 qwiik_jst

Commit message: Finalize PCB with Freerouting
Parts:
- S1, S10, S11, S12, S13, S14, S15, S16, S17, S18, S19, S2, S20, S21, S22, S23, S24, S25, S26, S27, S28, S29, S3, S4, S5, S6, S7, S8, S9: footprint scybin:switch_mx -> ceoloide:switch_mx
Routing:
- net SCL: track 33.3 -> 50.7 mm, vias 1 -> 2
- net R3: track 216.3 -> 233.6 mm, vias 8 -> 10
- net C4: track 215.9 -> 232.6 mm, vias 7 -> 6
- net C6: track 94.0 -> 108.7 mm, vias 2 -> 3
- net pinky_top_B: track 24.8 -> 38.3 mm
- net SDA: track 35.0 -> 46.1 mm
- net V+: track 42.6 -> 52.2 mm, vias 1 -> 3
- net C0: track 267.5 -> 259.7 mm, vias 4 -> 5
- net RST: track 181.1 -> 173.3 mm
- net C2: track 256.7 -> 263.2 mm, vias 7 -> 11
- net C3: track 237.5 -> 242.8 mm, vias 9 -> 7
- net R1: track 168.1 -> 172.8 mm, vias 9 -> 7
- net R2: track 195.6 -> 199.2 mm
- net C1: track 233.8 -> 230.3 mm, vias 5 -> 7
- net GND: track 244.6 -> 241.3 mm, vias 6 -> 5
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